Commit message: launching joint_state with mote_base, swapping LIDAR frame to match ROS conventions, adding maps but these should be removed after demo

File: mote_description/description/mote/robot.urdf (robot description, URDF)
Before this commit: robot mote, 6 links, 5 joints
Joints:
- joint laser_frame: origin xyz=0.0 0.0 0.1 rpy=0 0 0 -> xyz=0.0 0.0 0.1 rpy=0 0 3.14

Commit message: lowk hiwk making a mess of this branch and ima hate myself later BUT added maps and changed lidar frame to work

File: mote_description/description/mote/robot.urdf (robot description, URDF)
Before this commit: robot mote, 6 links, 5 joints
Joints:
- joint laser_frame: origin xyz=0.0 0.0 0.1 rpy=0 0 3.14 -> xyz=0.0 0.0 0.1 rpy=1.5708 0 3.1415

Commit message: fixing launch and package files removing deps removing maps

File: mote_description/description/mote/robot.urdf (robot description, URDF)
Before this commit: robot mote, 6 links, 5 joints
Joints:
- joint laser_frame: origin xyz=0.0 0.0 0.1 rpy=1.5708 0 3.1415 -> xyz=0.0 0.0 0.1 rpy=0 0 1.5705
