Commit message: Add onshape-to-robot support and import URDF

File: mote_description/description/mote/robot.urdf (robot description, URDF)
Before this commit: robot mote, 6 links, 5 joints
Links:
- removed link chassis
- removed link imu_link
- removed link laser
- removed link left_wheel_link
- removed link right_wheel_link
- added link imu, mass 1e-9
- added link lidar, mass 1e-9
- added link robot_body, mass 0.276245; collision mesh filename=package://mote_description/description/mote/assets/left_mot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; collision mesh filename=package://mote_description/description/mote/assets/left_mot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
- added link wheel_left, mass 0.0653752; collision mesh filename=package://mote_description/description/mote/assets/wheel_le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; visual mesh filename=package://mote_description/description/mote/assets/wheel_le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
- added link wheel_right, mass 0.0653752; collision mesh filename=package://mote_description/description/mote/assets/wheel_ri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; visual mesh filename=package://mote_description/description/mote/assets/wheel_ri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
- link base_link: mass None -> 1e-09
Joints:
- removed joint base_link_to_chassis
- removed joint laser_frame
- added joint base_link_to_robot_body: type fixed, parent base_link, child robot_body, origin xyz=0 0 0 rpy=0 -0 0, axis 0 0 1, limit effort=10 velocity=10
- added joint lidar_frame: type fixed, parent robot_body, child lidar, origin xyz=2.346e-09 -0.000467935 0.096 rpy=0 -0 0, axis 0 0 0
- joint imu_frame: axis (none) -> 0 0 0; child imu_link -> imu; origin xyz=0.0 0.0 0.0 rpy=0 0 0 -> xyz=2.669e-09 -0.000467935 0.0457 rpy=3.14159 -0 0; parent chassis -> robot_body
- joint left_wheel: child left_wheel_link -> wheel_left; limit effort=1 velocity=20 -> effort=10 velocity=10; origin xyz=0 0.075 0.033 rpy=-1.5707963267948966 0 0 -> xyz=2.669e-09 0.0493321 0.0325 rpy=-1.5708 1.30857 0; parent chassis -> robot_body
- joint right_wheel: child right_wheel_link -> wheel_right; limit effort=1 velocity=20 -> effort=10 velocity=10; origin xyz=0 -0.075 0.033 rpy=-1.5707963267948966 0 0 -> xyz=2.669e-09 -0.0502679 0.0325 rpy=1.5708 1.5675 3.14159; parent chassis -> robot_body
